File: PUTM_EV_IMD_SAFETY_2021.kicad_sch (KiCad schematic)
At the start: 61 parts, among them J1 MainConn, J2 SafetyConn, K1 FINDER-30.22.7.005.0010, Q1 2N7002, Q2 BSS138W-7-F, U1 SN74LS32D, U10 74LVC1G79, U2 MC78M12CDTG, U3 LM1117IMP-5.0, U4 LM393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

Commit message: changes of schematic components values
Parts:
- R15: value 47K -> 33K
- R21: value 0k -> 100k
- R22: value 0k -> 14.3k
Other:
- note removed: "0.5V"
- note removed: "2V"
Changed lines of the file:
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@@
-    (effects (font (size 1.27 1.27)) (justify left bottom))
-  )
-  (text "0.5V" (at 85.09 237.49 0)
     (effects (font (size 1.27 1.27)) (justify left bottom))
   )
@@
   (text "Connectors" (at 58.42 77.47 0)
     (effects (font (size 2.54 2.54)) (justify left bottom))
-  )
-  (text "2V" (at 85.09 229.87 0)
-    (effects (font (size 1.27 1.27)) (justify left bottom))
   )
   (text "Duty Check" (at 179.07 194.31 0)
@@
       (effects (font (size 1.27 1.27)) (justify right))
     )
-    (property "Value" "47K" (id 1) (at 93.218 241.173 0)
+    (property "Value" "33K" (id 1) (at 93.218 241.173 0)
       (effects (font (size 1.27 1.27)) (justify right))
     )
@@
       (effects (font (size 1.27 1.27)) (justify right))
     )
-    (property "Value" "0k" (id 1) (at 93.218 218.313 0)
+    (property "Value" "100k" (id 1) (at 93.218 218.313 0)
       (effects (font (size 1.27 1.27)) (justify right))
     )
@@
       (effects (font (size 1.27 1.27)) (justify right))
     )
-    (property "Value" "0k" (id 1) (at 93.218 225.933 0)
+    (property "Value" "14.3k" (id 1) (at 93.218 225.933 0)
       (effects (font (size 1.27 1.27)) (justify right))
     )
@@
     )
     (path "/00000000-0000-0000-0000-000061677e14"
-      (reference "R15") (unit 1) (value "47K") (footprint "Resistor_SMD:R_1206_3216Metric")
+      (reference "R15") (unit 1) (value "33K") (footprint "Resistor_SMD:R_1206_3216Metric")
     )
     (path "/00000000-0000-0000-0000-00006156bc00"
@@
     )
     (path "/00000000-0000-0000-0000-000062a6d899"
-      (reference "R21") (unit 1) (value "0k") (footprint "Resistor_SMD:R_1206_3216Metric")
+      (reference "R21") (unit 1) (value "100k") (footprint "Resistor_SMD:R_1206_3216Metric")
     )
     (path "/00000000-0000-0000-0000-000062aa6277"
-      (reference "R22") (unit 1) (value "0k") (footprint "Resistor_SMD:R_1206_3216Metric")
+      (reference "R22") (unit 1) (value "14.3k") (footprint "Resistor_SMD:R_1206_3216Metric")
     )
     (path "/00000000-0000-0000-0000-000062af5f32"
